File: 28ChFNIRS.sch (EAGLE design)
At the start: 134 parts, among them X1 332-50, X2 87758-4016

Commit message: Finished draft, time to test!
Connections:
- removed net N$46: D46.A
- net AOUT1: now also X2-8.S; no longer X2-17.S
- net AOUT10: now also X2-19.S; no longer X2-35.S
- net AOUT11: now also X2-23.S; no longer X2-37.S
- net AOUT12: now also X2-27.S; no longer X2-39.S
- net AOUT13: now also X2-31.S; no longer X2-2.S
- net AOUT14: now also X2-35.S; no longer X2-4.S
- net AOUT15: now also X2-4.S; no longer X2-6.S
- net AOUT16: now also X2-12.S; no longer X2-8.S
- net AOUT17: now also X2-18.S; no longer X2-10.S
- net AOUT18: now also X2-22.S; no longer X2-12.S
- net AOUT19: now also X2-26.S; no longer X2-14.S
- net AOUT2: now also X2-16.S; no longer X2-19.S
- net AOUT20: now also X2-30.S; no longer X2-16.S
- net AOUT21: now also X2-34.S; no longer X2-18.S
- net AOUT22: now also X2-2.S; no longer X2-20.S
- net AOUT23: now also X2-10.S; no longer X2-22.S
- net AOUT24: now also X2-17.S; no longer X2-24.S
- net AOUT25: now also X2-21.S; no longer X2-26.S
- net AOUT26: now also X2-25.S; no longer X2-28.S
- net AOUT27: now also X2-29.S; no longer X2-30.S
- net AOUT28: now also X2-33.S; no longer X2-32.S
- net AOUT3: now also X2-20.S; no longer X2-21.S
- net AOUT4: now also X2-24.S; no longer X2-23.S
- net AOUT5: now also X2-28.S; no longer X2-25.S
- net AOUT6: now also X2-32.S; no longer X2-27.S
- net AOUT7: now also X2-36.S; no longer X2-29.S
- net AOUT8: now also X2-6.S; no longer X2-31.S
- net AOUT9: now also X2-14.S; no longer X2-33.S
- net GND_ANA: no longer X2-34.S, X2-36.S, X2-38.S, X2-40.S
- net VLED10: now also X1-26.S; no longer X1-10.S
- net VLED11: now also X1-31.S; no longer X1-11.S
- net VLED12: now also X1-32.S; no longer X1-12.S
- net VLED13: now also X1-37.S; no longer X1-13.S
- net VLED14: now also X1-38.S; no longer X1-14.S
- net VLED15: now also X1-43.S; no longer X1-15.S
- net VLED16: now also X1-44.S; no longer X1-16.S
- net VLED17: now also X1-3.S; no longer X1-17.S
- net VLED18: now also X1-4.S; no longer X1-18.S
- net VLED19: now also X1-9.S; no longer X1-19.S
- net VLED20: now also X1-10.S; no longer X1-20.S
- net VLED21: now also X1-15.S; no longer X1-21.S
- net VLED22: now also X1-16.S; no longer X1-22.S
- net VLED23: now also X1-21.S; no longer X1-23.S
- net VLED24: now also X1-22.S; no longer X1-24.S
- net VLED25: now also X1-27.S; no longer X1-25.S
- net VLED26: now also X1-28.S; no longer X1-26.S
- net VLED27: now also X1-33.S; no longer X1-27.S
- net VLED28: now also X1-34.S; no longer X1-28.S
- net VLED29: now also X1-39.S; no longer X1-29.S
- net VLED3: now also X1-7.S; no longer X1-3.S
- net VLED30: now also X1-40.S; no longer X1-30.S
- net VLED31: now also X1-45.S; no longer X1-31.S
- net VLED32: now also X1-46.S; no longer X1-32.S
- net VLED33: now also X1-5.S; no longer X1-33.S
- net VLED34: now also X1-6.S; no longer X1-34.S
- net VLED35: now also X1-11.S; no longer X1-35.S
- net VLED36: now also X1-12.S; no longer X1-36.S
- net VLED37: now also X1-17.S; no longer X1-37.S
- net VLED38: now also X1-18.S; no longer X1-38.S
- net VLED39: now also X1-23.S; no longer X1-39.S
- net VLED4: now also X1-8.S; no longer X1-4.S
- net VLED40: now also X1-24.S; no longer X1-40.S
- net VLED41: now also X1-29.S; no longer X1-41.S
- net VLED42: now also X1-30.S; no longer X1-42.S
- net VLED43: now also X1-35.S; no longer X1-43.S
- net VLED44: now also X1-36.S; no longer X1-44.S
- net VLED45: now also X1-41.S; no longer X1-45.S
- net VLED46: now also D46.A, X1-42.S; no longer X1-46.S
- net VLED5: now also X1-13.S; no longer X1-5.S
- net VLED6: now also X1-14.S; no longer X1-6.S
- net VLED7: now also X1-19.S; no longer X1-7.S
- net VLED8: now also X1-20.S; no longer X1-8.S
- net VLED9: now also X1-25.S; no longer X1-9.S
