File: 28ChFNIRS.brd (EAGLE design)
At the start: 141.2 x 141.5 mm, 134 parts, among them X1 332-50, X2 87758-4016

Commit message: Finished draft, time to test!
Parts:
- moved SJ7 1.27 mm to (145.2, 27.9)
- moved SJ26 1.22 mm to (108.2, -44.4)
- moved SJ28 1.22 mm to (145.1, -44.9)
- moved SJ14 1.20 mm to (145.0, 3.81)
- moved SJ2 1.20 mm to (53.7, 28.1)
- moved SJ1 1.19 mm to (34.9, 27.8)
- moved SJ5 1.17 mm to (108.5, 27.7)
- moved SJ24 1.15 mm to (71.5, -45.0)
- moved SJ22 1.14 mm to (34.7, -44.9)
- moved SJ12 1.12 mm to (108.2, 3.91)
- moved SJ8 1.12 mm to (34.7, 4.34)
- moved SJ6 1.12 mm to (127.3, 27.9)
- moved SJ16 1.12 mm to (53.7, -20.8)
- moved SJ4 1.12 mm to (90.5, 28.0)
- moved SJ9 1.09 mm to (53.5, 3.63)
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Connections:
- removed net N$46: D46.A
- net AOUT1: now also X2.8; no longer X2.17
- net AOUT10: now also X2.19; no longer X2.35
- net AOUT11: now also X2.23; no longer X2.37
- net AOUT12: now also X2.27; no longer X2.39
- net AOUT13: now also X2.31; no longer X2.2
- net AOUT14: now also X2.35; no longer X2.4
- net AOUT15: now also X2.4; no longer X2.6
- net AOUT16: now also X2.12; no longer X2.8
- net AOUT17: now also X2.18; no longer X2.10
- net AOUT18: now also X2.22; no longer X2.12
- net AOUT19: now also X2.26; no longer X2.14
- net AOUT2: now also X2.16; no longer X2.19
- net AOUT20: now also X2.30; no longer X2.16
- net AOUT21: now also X2.34; no longer X2.18
- net AOUT22: now also X2.2; no longer X2.20
- net AOUT23: now also X2.10; no longer X2.22
- net AOUT24: now also X2.17; no longer X2.24
- net AOUT25: now also X2.21; no longer X2.26
- net AOUT26: now also X2.25; no longer X2.28
- net AOUT27: now also X2.29; no longer X2.30
- net AOUT28: now also X2.33; no longer X2.32
- net AOUT3: now also X2.20; no longer X2.21
- net AOUT4: now also X2.24; no longer X2.23
- net AOUT5: now also X2.28; no longer X2.25
- net AOUT6: now also X2.32; no longer X2.27
- net AOUT7: now also X2.36; no longer X2.29
- net AOUT8: now also X2.6; no longer X2.31
- net AOUT9: now also X2.14; no longer X2.33
- net GND_ANA: no longer X2.34, X2.36, X2.38, X2.40
- net VLED10: now also X1.26; no longer X1.10
- net VLED11: now also X1.31; no longer X1.11
- net VLED12: now also X1.32; no longer X1.12
- net VLED13: now also X1.37; no longer X1.13
- net VLED14: now also X1.38; no longer X1.14
- net VLED15: now also X1.43; no longer X1.15
- net VLED16: now also X1.44; no longer X1.16
- net VLED17: now also X1.3; no longer X1.17
- net VLED18: now also X1.4; no longer X1.18
- net VLED19: now also X1.9; no longer X1.19
- net VLED20: now also X1.10; no longer X1.20
- net VLED21: now also X1.15; no longer X1.21
- net VLED22: now also X1.16; no longer X1.22
- net VLED23: now also X1.21; no longer X1.23
- net VLED24: now also X1.22; no longer X1.24
- net VLED25: now also X1.27; no longer X1.25
- net VLED26: now also X1.28; no longer X1.26
- net VLED27: now also X1.33; no longer X1.27
- net VLED28: now also X1.34; no longer X1.28
- net VLED29: now also X1.39; no longer X1.29
- net VLED3: now also X1.7; no longer X1.3
- net VLED30: now also X1.40; no longer X1.30
- net VLED31: now also X1.45; no longer X1.31
- net VLED32: now also X1.46; no longer X1.32
- net VLED33: now also X1.5; no longer X1.33
- net VLED34: now also X1.6; no longer X1.34
- net VLED35: now also X1.11; no longer X1.35
- net VLED36: now also X1.12; no longer X1.36
- net VLED37: now also X1.17; no longer X1.37
- net VLED38: now also X1.18; no longer X1.38
- net VLED39: now also X1.23; no longer X1.39
- net VLED4: now also X1.8; no longer X1.4
- net VLED40: now also X1.24; no longer X1.40
- net VLED41: now also X1.29; no longer X1.41
- net VLED42: now also X1.30; no longer X1.42
- net VLED43: now also X1.35; no longer X1.43
- net VLED44: now also X1.36; no longer X1.44
- net VLED45: now also X1.41; no longer X1.45
- net VLED46: now also D46.A, X1.42; no longer X1.46
- net VLED5: now also X1.13; no longer X1.5
- net VLED6: now also X1.14; no longer X1.6
- net VLED7: now also X1.19; no longer X1.7
- net VLED8: now also X1.20; no longer X1.8
- net VLED9: now also X1.25; no longer X1.9
Routing:
- net GND_DIG: track 596.6 -> 940.6 mm, vias 0 -> 11
- net VLED46: track 1.60 -> 72.9 mm
- net AOUT28: track 23.1 -> 86.3 mm, vias 0 -> 1
- net AOUT14: track 73.1 -> 135.4 mm, vias 0 -> 1
- net VLED15: track 84.1 -> 144.7 mm
- net AOUT21: track 46.6 -> 107.0 mm, vias 0 -> 1
- net VLED16: track 79.2 -> 139.0 mm
- net VLED31: track 58.3 -> 117.5 mm
- net VLED32: track 53.6 -> 111.9 mm
- net VLED47: track 31.6 -> 89.5 mm
- net VLED48: track 26.5 -> 83.6 mm
- net AOUT7: track 100.3 -> 156.1 mm, vias 0 -> 1
- net AOUT27: track 23.0 -> 74.7 mm, vias 0 -> 1
- net AOUT13: track 72.3 -> 122.2 mm, vias 0 -> 1
- net AOUT20: track 47.4 -> 95.8 mm, vias 0 -> 1
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Other:
- board text added: "1"
- board text added: "10"
- board text added: "11"
- board text added: "12"
- board text added: "13"
- board text added: "14"
- board text added: "15"
- board text added: "16"
- board text added: "17"
- board text added: "18"
- board text added: "19"
- board text added: "2"
- board text added: "20"
- board text added: "21"
- board text added: "22"
- board text added: "23"
- board text added: "24"
- board text added: "25"
- board text added: "26"
- board text added: "27"
- board text added: "28"
- board text added: "28 optical channels, 24 LED pairs"
- board text added: "29"
- board text added: "3"
- board text added: "30"
- board text added: "31"
- board text added: "32"
- board text added: "33"
- board text added: "34"
- board text added: "35"
- board text added: "36"
- board text added: "37"
- board text added: "38"
- board text added: "39"
- board text added: "4"
- board text added: "40"
- board text added: "41"
- board text added: "42"
- board text added: "43"
- board text added: "44"
- board text added: "45"
- board text added: "46"
- board text added: "47"
- board text added: "48"
- board text added: "5"
- board text added: "6"
- board text added: "7"
- board text added: "8"
- board text added: "9"
- board text added: "A1"
- board text added: "A10"
- board text added: "A11"
- board text added: "A12"
- board text added: "A13"
- board text added: "A14"
- board text added: "A15"
- board text added: "A16"
- board text added: "A17"
- board text added: "A18"
- board text added: "A19"
- board text added: "A2"
- board text added: "A20"
- board text added: "A21"
- board text added: "A22"
- board text added: "A23"
- board text added: "A24"
- board text added: "A25"
- board text added: "A26"
- board text added: "A27"
- board text added: "A28"
- board text added: "A3"
- board text added: "A4"
- board text added: "A5"
- board text added: "A6"
- board text added: "A7"
- board text added: "A8"
- board text added: "A9"
- board text added: "BASED ON pnas.org/content/104/29/12169"
- board text added: "DIY DIFFUSE OPTICAL TOMOGRAPHY"
- board text added: "G_A"
- board text added: "G_D"
- board text added: "JOSHUA BREWSTER (MIT LICENSE)"
- board text added: "LEDs"
- board text added: "NC"
- board text added: "SENSORS"
- board text added: "The Dream Machine The "2Kool4Skool" The "End of Privacy""
- board text added: "Use OPT101 (the cheap aliexpress ones) and 1206 spec LEDs"
- board text added: "V_A"

Commit message: added a few mounting holes
Routing:
- net GND_DIG: track 940.6 -> 939.8 mm
Changed lines of the file:
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@@
 <text x="61.6712" y="-91.4908" size="0.6096" layer="27">18</text>
 <text x="59.9186" y="-91.4654" size="0.6096" layer="27">2</text>
-<text x="56.4134" y="-90.3224" size="0.6096" layer="27">LEDs</text>
-<text x="56.388" y="-97.79" size="0.6096" layer="27">LEDs</text>
+<text x="56.1594" y="-92.9132" size="0.6096" layer="27">LEDs</text>
+<text x="56.1848" y="-95.0722" size="0.6096" layer="27">LEDs</text>
 <text x="105.5878" y="-78.5876" size="0.6096" layer="27" rot="R90">SENSORS</text>
 <text x="63.4746" y="-78.5368" size="0.6096" layer="27" rot="R90">SENSORS</text>
@@
 The "2Kool4Skool"
 The "End of Privacy"</text>
+<hole x="15.8496" y="34.8742" drill="2.54"/>
+<hole x="152.2222" y="35.1536" drill="2.54"/>
+<hole x="111.3028" y="-97.7392" drill="2.54"/>
+<hole x="57.4802" y="-97.7646" drill="2.54"/>
+<hole x="20.193" y="39.243" drill="2.54"/>
+<hole x="148.1328" y="39.3954" drill="2.54"/>
+<circle x="57.4802" y="-97.7646" radius="1.37535625" width="0.2032" layer="101"/>
+<circle x="57.4802" y="-97.79" radius="1.380271875" width="0.2032" layer="100"/>
+<circle x="111.3028" y="-97.7392" radius="1.380271875" width="0.2032" layer="100"/>
+<circle x="111.3028" y="-97.7392" radius="1.37535625" width="0.2032" layer="101"/>
 </plain>
 <attributes>
@@
 </element>
 <element name="D5" library="epic" package="LED-1206" value="" x="56.1086" y="17.0688" smashed="yes">
-<attribute name="NAME" x="48.9966" y="16.1798" size="1.778" layer="25" font="vector"/>
+<attribute name="NAME" x="48.9966" y="16.3322" size="1.778" layer="25" font="vector"/>
 <attribute name="VALUE" x="53.5686" y="13.7668" size="1.778" layer="27" font="vector"/>
 </element>
@@
 <wire x1="149.7598" y1="-31.5214" x2="149.7598" y2="-33.7312" width="0.508" layer="1"/>
 <wire x1="149.7598" y1="-33.7312" x2="149.7598" y2="-34.8756" width="0.508" layer="1"/>
-<wire x1="149.7598" y1="-34.8756" x2="150.622" y2="-35.7378" width="0.508" layer="1"/>
+<wire x1="149.7598" y1="-34.8756" x2="150.2156" y2="-35.3314" width="0.508" layer="1"/>
 <wire x1="20.9818" y1="-51.7666" x2="52.2224" y2="-83.0072" width="0.508" layer="1"/>
 <via x="40.132" y="-58.1914" extent="1-16" drill="0.35"/>
@@
 <via x="119.1006" y="-75.0062" extent="1-16" drill="0.35"/>
 <wire x1="131.7498" y1="-35.3568" x2="131.7498" y2="-62.357" width="0.508" layer="1"/>
-<wire x1="150.622" y1="-57.45766875" x2="113.35366875" y2="-94.726" width="0.508" layer="1"/>
-<wire x1="109.7788" y1="-94.726" x2="113.35366875" y2="-94.726" width="0.508" layer="1"/>
-<wire x1="150.622" y1="-35.7378" x2="150.622" y2="-57.45766875" width="0.508" layer="1"/>
+<wire x1="150.2156" y1="-57.05126875" x2="112.54086875" y2="-94.726" width="0.508" layer="1"/>
+<wire x1="109.7788" y1="-94.726" x2="112.54086875" y2="-94.726" width="0.508" layer="1"/>
+<wire x1="150.2156" y1="-35.3314" x2="150.2156" y2="-57.05126875" width="0.508" layer="1"/>
 <wire x1="108.077" y1="-74.9046" x2="108.1024" y2="-74.93" width="0.508" layer="16"/>
 <wire x1="108.1024" y1="-74.93" x2="108.1024" y2="-85.8774" width="0.508" layer="16"/>
