File: 16ChFNIRS.sch (EAGLE design)
At the start: 68 parts

Commit message: edit jumpers
Parts:
- SJ1, SJ10, SJ11, SJ12, SJ13, SJ14, SJ15, SJ2, SJ22, SJ3, SJ4, SJ5, SJ6, SJ7, SJ8, SJ9: value SOLDERJUMPERNC -> (none); device headers:SOLDERJUMPERNC -> jumper:SJ
