File: 16ChFNIRS.brd (EAGLE design)
At the start: 198.4 x 48.5 mm, 68 parts

Commit message: edit jumpers
Parts:
- SJ1, SJ10, SJ11, SJ12, SJ13, SJ14, SJ15, SJ2, SJ22, SJ3, SJ4, SJ5, SJ6, SJ7, SJ8, SJ9: value SOLDERJUMPERNC -> (none); device headers:SJ_2S_SMALL -> jumper:SJ

Commit message: fix
Routing:
- net AOUT15: track 199.4 -> 200.0 mm
